Commit message: add a1 env gazebo

File: OmniIsaacGymEnvs/unitree_ws/src/unitree_ros/robots/a1_description/urdf/a1.urdf (robot description, URDF)
Before this commit: robot a1, 23 links, 22 joints
Links:
- added link camera_link, mass 0.001; collision box size=1.001 1.001 1.001; visual box size=0.001 0.001 0.001
Joints:
- added joint camera_joint: type fixed, parent trunk, child camera_link, origin xyz=0 0 0 rpy=0 0 0

File: OmniIsaacGymEnvs/unitree_ws/src/unitree_ros/robots/a1_description/xacro/gazebo.xacro (robot description, xacro)
@@ -55,4 +55,53 @@
         </sensor>
     </gazebo>
+      <gazebo reference="camera_link">
+  <sensor type="camera" name="ab_camera">
+      <always_on>true</always_on>
+      <update_rate>20</update_rate>
+      <visualize>true</visualize>
+      <camera name="ab_camera">
+        <horizontal_fov>1.2</horizontal_fov>
+        <image>
+          <format>R8G8B8</format>
+          <width>800</width>
+          <height>600</height>
+        </image>
+        <clip>
+          <near>0.02</near>
+          <far>300</far>
+        </clip>
+        <noise>
+          <type>gaussian</type>
+          <mean>0.0</mean>
+          <stddev>0.007</stddev>
+        </noise>
+        <distortion>
+          <k1>-0.25</k1>
+          <k2>0.12</k2>
+          <k3>0.0</k3>
+          <p1>0.0</p1>
+          <p2>0.0</p2>
+          <center>0.5 0.5</center>
+        </distortion>
+      </camera>
+      <plugin name="camera_controller" filename="libgazebo_ros_camera.so">
+        <imageTopicName>/ab_camera/image_raw</imageTopicName>
+        <cameraInfoTopicName>/ab_camera/camera_info</cameraInfoTopicName>
+        <cameraName>camera1</cameraName>
+        <frameName>camera_link</frameName>
+        <updateRate>10.0</updateRate>
+        <CxPrime>0.0</CxPrime>
+        <Cx>0.0</Cx>
+        <Cy>0.0</Cy>
+        <focalLength>0.0</focalLength> <!-- use computed_focal_length -->
+        <hackBaseline>0.12</hackBaseline> <!-- use for P[3] -->
+        <distortionK1>0.05</distortionK1>
+        <distortionK2>-0.05</distortionK2>
+        <distortionK3>0.0</distortionK3>
+        <distortionT1>0.0</distortionT1>
+        <distortionT2>0.0</distortionT2>
+      </plugin>
+    </sensor>
+  </gazebo>
     <!-- Foot contacts. -->
     <gazebo reference="FR_calf">

File: OmniIsaacGymEnvs/unitree_ws/src/unitree_ros/robots/a1_description/xacro/robot.xacro (robot description, xacro)
@@ -110,4 +110,29 @@
         </collision>
     </link>
+    <joint name="camera_joint" type="fixed">
+        <parent link="trunk"/>
+        <child link="camera_link"/>
+        <origin rpy="0 1.57 0" xyz="0 0 -0.05"/>
+    </joint>
+    <link name="camera_link">
+        <inertial>
+            <mass value="0.001"/>
+            <origin rpy="0 0 0" xyz="0 0 0"/>
+            <inertia ixx="0.0001" ixy="0" ixz="0" iyy="0.0001" iyz="0" izz="0.0001"/>
+        </inertial>
+        <visual>
+            <origin rpy="0 0 0" xyz="0 0 0"/>
+            <geometry>
+                <box size="0.001 0.001 0.001"/>
+            </geometry>
+            <material name="red"/>
+        </visual>
+        <collision>
+            <origin rpy="0 0 0" xyz="0 0 0"/>
+            <geometry>
+                <box size=".001 .001 .001"/>
+            </geometry>
+        </collision>
+    </link>
     <xacro:leg name="FR" mirror="-1" mirror_dae="False" front_hind="1" front_hind_dae="True">
         <origin rpy="0 0 0" xyz="${leg_offset_x} ${-leg_offset_y} 0"/>
