Commit message: add beam

File: OmniIsaacGymEnvs/unitree_ws/src/unitree_ros/robots/a1_description/xacro/gazebo.xacro (robot description, xacro)
@@ -64,6 +64,6 @@
         <image>
           <format>R8G8B8</format>
-          <width>800</width>
-          <height>600</height>
+          <width>1280</width>
+          <height>720</height>
         </image>
         <clip>

File: OmniIsaacGymEnvs/unitree_ws/src/unitree_ros/robots/a1_description/xacro/robot.xacro (robot description, xacro)
@@ -113,5 +113,5 @@
         <parent link="trunk"/>
         <child link="camera_link"/>
-        <origin rpy="0 1.57 0" xyz="0 0 -0.05"/>
+        <origin rpy="0 1.57 0" xyz="0.04 0 -0.05"/>
     </joint>
     <link name="camera_link">
